File: BUCK_LMR33630/BUCK_LMR33630.kicad_sch (KiCad schematic)
At the start: 13 parts, among them U1 LMR33630ADDA

Commit message: Update doc
Parts:
- removed C9: 22uF, Capacitor_SMD:C_1206_3216Metric, symbol Device:C
- added H1, H2, H3, H4: MountingHole, MountingHole:MountingHole_3.2mm_M3, symbol Mechanical:MountingHole
- added J1, J2: Conn_01x02, TerminalBlock_Phoenix:TerminalBlock_Phoenix_MKDS-1,5-2-5.08_1x02_P5.08mm_Horizontal, symbol Connector_Generic:Conn_01x02
- C1: value CP -> 10uF; footprint (none) -> Capacitor_SMD:C_1206_3216Metric_Pad1.33x1.80mm_HandSolder; symbol LMR33630_REG-rescue:CP-Device -> Device:C
- C2: value C_Small -> 220nF; footprint (none) -> Capacitor_SMD:C_1206_3216Metric_Pad1.33x1.80mm_HandSolder
- C4: value C_Small -> 100nF; footprint (none) -> Capacitor_SMD:C_1206_3216Metric_Pad1.33x1.80mm_HandSolder
- C6, C7, C8: footprint Capacitor_SMD:C_1206_3216Metric -> Capacitor_SMD:C_1206_3216Metric_Pad1.33x1.80mm_HandSolder
- L1: footprint (none) -> Inductor_SMD:L_Bourns-SRU1028_10.0x10.0mm; MF (none) -> BOURNS; MPN (none) -> SRU1048-6R8Y
- U1: MF (none) -> TEXAS INSTRUMENTS; MPN (none) -> LMR33630ADDA
Connections:
- net GND: now also J1.2 (Pin_2), J2.1 (Pin_1)
- net VIN: now also J1.1 (Pin_1)
- net VOUT: now also J2.2 (Pin_2)
Other:
- company: (none) -> Jairo Estefanía
- title: (none) -> BUCK_LMR3360
